File: hardware/v1.0/icepi-zero.kicad_pcb (KiCad board)
At the start: 4 copper layers, 65 x 30 mm, 138 parts, among them J1 Conn_02x20_Counter_Clockwise, J2 HDMI_C_1.3, J3 USB_C_Receptacle_USB2.0_14P, J4 USB_C_Receptacle_USB2.0_14P, J5 USB_C_Receptacle_USB2.0_14P, J6 Micro_SD_Card_Det2, SW1 SW_Push, U1 ECP5U_12_CABGA256, U10 W9825G6KH, U11 W25Q128JVS, U2 TLV62569DBV, U3 TLV62569DBV, U4 TLV62569DBV, U5 PCA9306DC1, U6 FT231XQ, U7 TPD2EUSB30A, U8 TPD2EUSB30A, U9 TPD2EUSB30A, Y1 SITxxxxxx-1x-33E-50.000000

Commit message: Increase pad spacing to 1.9mm and change SCL name to SCK
Connections:
- J2 pad 15: /GPIO/GPDI_SCK -> /GPIO/GPDI_SCK_5V
- J2 pad 16: GPDI_SDA -> /GPIO/GPDI_SDA_5V
- R16 pad 2: GPDI_SCL -> /GPIO/GPDI_SCK_5V
- R17 pad 2: GPDI_SDA -> /GPIO/GPDI_SDA_5V
- R19 pad 2: /GPIO/GPDI_SCK -> GPDI_SCK
- U1 pad T3: GPDI_SCL -> GPDI_SCK
- U5 pad 3: /GPIO/GPDI_SCK -> GPDI_SCK
- U5 pad 5: GPDI_SDA -> /GPIO/GPDI_SDA_5V
- U5 pad 6: GPDI_SCL -> /GPIO/GPDI_SCK_5V
Routing:
- net GPDI_SCL: track 48.2 -> 0.00 mm, vias 4 -> 0
- net GPDI_SCK: track 0.00 -> 37.6 mm, vias 0 -> 2
- net /GPIO/GPDI_SCK_5V: track 0.00 -> 10.5 mm, vias 0 -> 2
- net GPDI_SDA: track 44.9 -> 37.9 mm
- net /GPIO/GPDI_SDA_5V: track 0.00 -> 7.01 mm
