File: hardware/v1.2/flash.kicad_sch (KiCad schematic)
At the start: 14 parts, among them J6 Micro_SD_Card_Det2, U1 ECP5U_25F_CABGA256, U11 W25Q128JVS

Commit message: Trying to document my journey :)
Parts:
- renumbered R31 to R43, R32 to R44, R33 to R45, R34 to R46, R35 to R47, R36 to R48, R37 to R49, R38 to R50
Changed lines of the file:
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@@
 		(on_board yes)
 		(dnp no)
-		(property "Reference" "R36"
+		(property "Reference" "R48"
 			(at 103.632 64.77 90)
 			(effects
@@
 			(project "icepi-zero"
 				(path "/f88da08e-cf42-4d03-a08f-3f602fe6658d/d4e07380-5584-4eac-bd07-d260a33e64d7"
-					(reference "R36")
+					(reference "R48")
 					(unit 1)
 				)
@@
 		(on_board yes)
 		(dnp no)
-		(property "Reference" "R37"
+		(property "Reference" "R49"
 			(at 109.982 64.77 90)
 			(effects
@@
 			(project "icepi-zero"
 				(path "/f88da08e-cf42-4d03-a08f-3f602fe6658d/d4e07380-5584-4eac-bd07-d260a33e64d7"
-					(reference "R37")
+					(reference "R49")
 					(unit 1)
 				)
@@
 		(on_board yes)
 		(dnp no)
-		(property "Reference" "R34"
+		(property "Reference" "R46"
 			(at 85.852 64.77 90)
 			(effects
@@
 			(project "icepi-zero"
 				(path "/f88da08e-cf42-4d03-a08f-3f602fe6658d/d4e07380-5584-4eac-bd07-d260a33e64d7"
-					(reference "R34")
+					(reference "R46")
 					(unit 1)
 				)
@@
 		(on_board yes)
 		(dnp no)
-		(property "Reference" "R38"
+		(property "Reference" "R50"
 			(at 116.332 64.77 90)
 			(effects
@@
 			(project "icepi-zero"
 				(path "/f88da08e-cf42-4d03-a08f-3f602fe6658d/d4e07380-5584-4eac-bd07-d260a33e64d7"
-					(reference "R38")
+					(reference "R50")
 					(unit 1)
 				)
@@
 		(on_board yes)
 		(dnp no)
-		(property "Reference" "R31"
+		(property "Reference" "R43"
 			(at 66.802 64.77 90)
 			(effects
@@
 			(project "icepi-zero"
 				(path "/f88da08e-cf42-4d03-a08f-3f602fe6658d/d4e07380-5584-4eac-bd07-d260a33e64d7"
-					(reference "R31")
+					(reference "R43")
 					(unit 1)
 				)
@@
 		(on_board yes)
 		(dnp no)
-		(property "Reference" "R32"
+		(property "Reference" "R44"
 			(at 73.152 64.77 90)
 			(effects
@@
 			(project "icepi-zero"
 				(path "/f88da08e-cf42-4d03-a08f-3f602fe6658d/d4e07380-5584-4eac-bd07-d260a33e64d7"
-					(reference "R32")
+					(reference "R44")
 					(unit 1)
 				)
@@
 		(on_board yes)
 		(dnp no)
-		(property "Reference" "R35"
+		(property "Reference" "R47"
 			(at 92.202 64.77 90)
 			(effects
@@
 			(project "icepi-zero"
 				(path "/f88da08e-cf42-4d03-a08f-3f602fe6658d/d4e07380-5584-4eac-bd07-d260a33e64d7"
-					(reference "R35")
+					(reference "R47")
 					(unit 1)
 				)
@@
 		(on_board yes)
 		(dnp no)
-		(property "Reference" "R33"
+		(property "Reference" "R45"
 			(at 79.502 64.77 90)
 			(effects
@@
 			(project "icepi-zero"
 				(path "/f88da08e-cf42-4d03-a08f-3f602fe6658d/d4e07380-5584-4eac-bd07-d260a33e64d7"
-					(reference "R33")
-					(unit 1)
-				)
+					(reference "R45")
+					(unit 1)
+				)
