File: hardware/v1.2/usb.kicad_sch (KiCad schematic)
At the start: 47 parts, among them J3 USB_C_Receptacle_USB2.0_14P, J4 USB_C_Receptacle_USB2.0_14P, J5 USB_C_Receptacle_USB2.0_14P, U1 ECP5-CABGA256, U6 FT231XQ, U7 TPD2EUSB30A, U8 TPD2EUSB30A, U9 TPD2EUSB30A

Commit message: Newest source files
Other:
- moved on the sheet: D13, D14, R41, R42
Changed lines of the file:
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@@
 	)
 	(junction
-		(at 97.79 185.42)
+		(at 96.52 185.42)
 		(diameter 0)
 		(color 0 0 0 0)
@@
 	)
 	(junction
-		(at 119.38 185.42)
+		(at 118.11 185.42)
 		(diameter 0)
 		(color 0 0 0 0)
@@
 	(wire
 		(pts
-			(xy 118.11 187.96) (xy 119.38 187.96)
+			(xy 116.84 187.96) (xy 118.11 187.96)
 		)
 		(stroke
@@
 	(wire
 		(pts
-			(xy 97.79 182.88) (xy 99.06 182.88)
+			(xy 96.52 182.88) (xy 97.79 182.88)
 		)
 		(stroke
@@
 	(wire
 		(pts
-			(xy 119.38 185.42) (xy 135.89 185.42)
+			(xy 118.11 185.42) (xy 135.89 185.42)
 		)
 		(stroke
@@
 	(wire
 		(pts
-			(xy 92.71 185.42) (xy 97.79 185.42)
+			(xy 90.17 185.42) (xy 96.52 185.42)
 		)
 		(stroke
@@
 	(wire
 		(pts
-			(xy 119.38 185.42) (xy 119.38 187.96)
+			(xy 118.11 185.42) (xy 118.11 187.96)
 		)
 		(stroke
@@
 	(wire
 		(pts
-			(xy 97.79 187.96) (xy 99.06 187.96)
+			(xy 96.52 187.96) (xy 97.79 187.96)
 		)
 		(stroke
@@
 	(wire
 		(pts
-			(xy 106.68 187.96) (xy 110.49 187.96)
+			(xy 105.41 187.96) (xy 109.22 187.96)
 		)
 		(stroke
@@
 	(wire
 		(pts
-			(xy 97.79 187.96) (xy 97.79 185.42)
+			(xy 96.52 187.96) (xy 96.52 185.42)
 		)
 		(stroke
@@
 	(wire
 		(pts
-			(xy 118.11 182.88) (xy 119.38 182.88)
+			(xy 116.84 182.88) (xy 118.11 182.88)
 		)
 		(stroke
@@
 	(wire
 		(pts
-			(xy 106.68 182.88) (xy 110.49 182.88)
+			(xy 105.41 182.88) (xy 109.22 182.88)
 		)
 		(stroke
@@
 	(wire
 		(pts
-			(xy 119.38 182.88) (xy 119.38 185.42)
+			(xy 118.11 182.88) (xy 118.11 185.42)
 		)
 		(stroke
@@
 	(wire
 		(pts
-			(xy 97.79 185.42) (xy 97.79 182.88)
+			(xy 96.52 185.42) (xy 96.52 182.88)
 		)
 		(stroke
@@
 	)
 	(label "D0+"
-		(at 92.71 185.42 0)
+		(at 90.17 185.42 0)
 		(effects
 			(font
@@
 	(symbol
 		(lib_id "Diode:1N914WT")
-		(at 114.3 182.88 0)
+		(at 113.03 182.88 0)
 		(mirror x)
 		(unit 1)
@@
 		(dnp no)
 		(property "Reference" "D13"
-			(at 114.3 176.53 0)
+			(at 113.03 176.53 0)
 			(effects
 				(font
@@
 		)
 		(property "Value" "1N914WT"
-			(at 114.3 179.07 0)
+			(at 113.03 179.07 0)
 			(effects
 				(font
@@
 		)
 		(property "Footprint" "Diode_SMD:D_SOD-523"
-			(at 114.3 178.435 0)
+			(at 113.03 178.435 0)
 			(effects
 				(font
@@
 		)
 		(property "Datasheet" "http://www.mouser.com/ds/2/149/1N4148WT-461550.pdf"
-			(at 114.3 182.88 0)
+			(at 113.03 182.88 0)
 			(effects
 				(font
@@
 		)
 		(property "Description" "75V 0.15A Fast switching Diode, SOD-523"
-			(at 114.3 182.88 0)
+			(at 113.03 182.88 0)
 			(effects
 				(font
@@
 		)
 		(property "Sim.Device" "D"
-			(at 114.3 182.88 0)
+			(at 113.03 182.88 0)
 			(effects
 				(font
@@
 		)
 		(property "Sim.Pins" "1=K 2=A"
-			(at 114.3 182.88 0)
+			(at 113.03 182.88 0)
 			(effects
 				(font
@@
 		)
 		(property "LCSC Part #" "C2836064"
-			(at 114.3 182.88 0)
+			(at 113.03 182.88 0)
 			(effects
 				(font
@@
 	(symbol
 		(lib_id "Diode:1N914WT")
-		(at 114.3 187.96 0)
+		(at 113.03 187.96 0)
 		(mirror y)
 		(unit 1)
@@
 		(dnp no)
 		(property "Reference" "D14"
-			(at 114.3 194.31 0)
+			(at 113.03 194.31 0)
 			(effects
 				(font
@@
 		)
 		(property "Value" "1N914WT"
-			(at 114.3 191.77 0)
+			(at 113.03 191.77 0)
 			(effects
 				(font
@@
 		)
 		(property "Footprint" "Diode_SMD:D_SOD-523"
-			(at 114.3 192.405 0)
+			(at 113.03 192.405 0)
 			(effects
 				(font
@@
 		)
 		(property "Datasheet" "http://www.mouser.com/ds/2/149/1N4148WT-461550.pdf"
-			(at 114.3 187.96 0)
+			(at 113.03 187.96 0)
 			(effects
 				(font
@@
 		)
 		(property "Description" "75V 0.15A Fast switching Diode, SOD-523"
-			(at 114.3 187.96 0)
+			(at 113.03 187.96 0)
 			(effects
 				(font
@@
 		)
 		(property "Sim.Device" "D"
-			(at 114.3 187.96 0)
+			(at 113.03 187.96 0)
 			(effects
 				(font
@@
 		)
 		(property "Sim.Pins" "1=K 2=A"
-			(at 114.3 187.96 0)
+			(at 113.03 187.96 0)
 			(effects
 				(font
@@
 		)
 		(property "LCSC Part #" "C2836064"
-			(at 114.3 187.96 0)
+			(at 113.03 187.96 0)
 			(effects
 				(font
@@
 	(symbol
 		(lib_id "Device:R")
-		(at 102.87 187.96 270)
+		(at 101.6 187.96 270)
 		(unit 1)
 		(exclude_from_sim no)
@@
 		(dnp no)
 		(property "Reference" "R42"
-			(at 102.87 190.246 90)
+			(at 101.6 190.246 90)
 			(effects
 				(font
@@
 		)
 		(property "Value" "15k"
-			(at 102.87 187.96 90)
+			(at 101.6 187.96 90)
 			(effects
 				(font
@@
 		)
 		(property "Footprint" "Resistor_SMD:R_0402_1005Metric"
-			(at 102.87 186.182 90)
+			(at 101.6 186.182 90)
 			(effects
 				(font
@@
 		)
 		(property "Datasheet" "~"
-			(at 102.87 187.96 0)
+			(at 101.6 187.96 0)
 			(effects
 				(font
@@
 		)
 		(property "Description" "Resistor"
-			(at 102.87 187.96 0)
+			(at 101.6 187.96 0)
 			(effects
 				(font
@@
 		)
 		(property "LCSC Part #" "C25756"
-			(at 102.87 187.96 0)
+			(at 101.6 187.96 0)
 			(effects
 				(font
@@
 	(symbol
 		(lib_id "Device:R")
-		(at 102.87 182.88 270)
+		(at 101.6 182.88 270)
 		(mirror x)
 		(unit 1)
@@
 		(dnp no)
 		(property "Reference" "R41"
-			(at 102.87 180.594 90)
+			(at 101.6 180.594 90)
 			(effects
 				(font
@@
 		)
 		(property "Value" "1k"
-			(at 102.87 182.88 90)
+			(at 101.6 182.88 90)
 			(effects
 				(font
@@
 		)
 		(property "Footprint" "Resistor_SMD:R_0402_1005Metric"
-			(at 102.87 184.658 90)
+			(at 101.6 184.658 90)
 			(effects
 				(font
@@
 		)
 		(property "Datasheet" "~"
-			(at 102.87 182.88 0)
+			(at 101.6 182.88 0)
 			(effects
 				(font
@@
 		)
 		(property "Description" "Resistor"
-			(at 102.87 182.88 0)
+			(at 101.6 182.88 0)
 			(effects
 				(font
@@
 		)
 		(property "LCSC Part #" "C11702"
-			(at 102.87 182.88 0)
+			(at 101.6 182.88 0)
 			(effects
 				(font
