File: hardware/v1.3/icepi-zero.kicad_pcb (KiCad board)
At the start: 4 copper layers, 65 x 30 mm, 165 parts, among them J1 Conn_02x20_Counter_Clockwise, J2 GPDI_C_1.3, J3 USB_C_Receptacle_USB2.0_14P, J4 USB_C_Receptacle_USB2.0_14P, J5 USB_C_Receptacle_USB2.0_14P, J6 Micro_SD_Card_Det2, SW1 SW_Push, SW2 SW_Push, U1 ECP5-CABGA256, U10 TPD2EUSB30A, U11 W9825G6KH, U12 W25Q128JVS, U2 TLV62569DBV, U3 TLV62569DBV, U4 TLV62569DBV, U5 TPD2EUSB30A, U6 PCA9306DC1, U7 TPD2EUSB30A, U8 TPD2EUSB30A, U9 FT231XQ, Y1 SG-8018CG 50.000000MHz

Commit message: Change LED's resistor values to make them dimmer
Parts:
- removed REF**: UKCA-Logo_6x6mm_SilkScreen, Symbol:UKCA-Logo_6x6mm_SilkScreen
- removed REF**: CE-Logo_8.5x6mm_SilkScreen, Symbol:CE-Logo_8.5x6mm_SilkScreen
- L1, L2, L3: value 2.2uH 100mA+ 400mO- -> 2.2uH
- R1, R2, R3, R4, R5: value 470 -> 1k
Connections:
- net DONE renamed /Flash/DONE
- net INITN renamed /Flash/INITN
- net PROGRAMMING renamed /Flash/PROGRAMMING
